Commit message: update urdf

File: robot_model/mp_500/mp_500.urdf (robot description, URDF)
Before this commit: robot mp_500, 6 links, 5 joints
Links:
- link base_footprint: geometry collision mesh filename=package://neo_mp_500-2/robot_model/mp_500/meshes/MP-500-BOD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 scale=0.001 0.001 0.001; visual mesh filename=package://neo_mp_500-2/robot_model/mp_500/meshes/MP-500-BOD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 scale=0.001 0.001 0.001
- link wheel_right_link: geometry collision mesh filename=package://neo_mp_500-2/robot_model/mp_500/meshes/MP-500-WHE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 scale=0.001 0.001 0.001; visual mesh filename=package://neo_mp_500-2/robot_model/mp_500/meshes/MP-500-WHE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 scale=0.001 0.001 0.001
Joints:
- joint wheel_left_joint: type revolute -> fixed
- joint wheel_right_joint: type revolute -> fixed
